File: pcb/compass-controller/compass-controller.kicad_pcb (KiCad board)
At the start: 2 copper layers, 209 parts, among them J101 USB_C_Receptacle_USB2.0_16P, J102 USB5V, J103 Barrel_Jack, J104 TC2030, J105 STLINK, J106 LEFT BUTTON, J107 LEFT BUTTON, J108 Micro_SD_Card, J109 TFT DISPLAY, J110 ENCODER BUTTON, J111 ENCODER, J201 LIM, J202 HOMING, J203 MOTOR, J301 LIM, J302 HOMING, J303 MOTOR, J401 LIM, J402 HOMING, J403 MOTOR, J501 RJ45_Shielded, J601 RJ45_Shielded, J701 RJ45_Shielded, J801 RJ45_Shielded, Q501 AO3401A, Q601 AO3401A, Q701 AO3401A, Q801 AO3401A, SW101 TS1187, SW102 TS1187, U101 STM32G431CBUx, U102 LTV-247, U103 TPS5430DDA, U104 TPSPX3819M5-L-3-3, U201 TMC2209, U301 TMC2209, U401 TMC2209, U501 TXU0304RUTR, U601 TXU0304RUTR, U701 TXU0304RUTR, U801 TXU0304RUTR, Y101 12MHz

Commit message: work on layout
Parts:
- removed R113: 0R, Resistor_SMD:R_0603_1608Metric
- removed R118: 5k1, Resistor_SMD:R_0603_1608Metric
- J107: value LEFT BUTTON -> RIGHT BUTTON
- moved C101 198.5 mm to (213.7, 88.1), turned to 180 degrees
- moved R101 193.7 mm to (213.8, 89.8), turned to 180 degrees
- moved R102 191.8 mm to (213.7, 86.5), turned to 180 degrees
- moved R103 190.3 mm to (213.7, 83.5), turned to 180 degrees
- moved H101 186.2 mm to (196.3, 68.8)
- moved R119 177.6 mm to (185.9, 121.5), turned to -90 degrees
- moved C110 174.2 mm to (186.9, 105.3), turned to -90 degrees
- moved C117 173.1 mm to (183.8, 105.3), turned to -90 degrees
- moved H102 172.6 mm to (196.3, 128.8)
- moved R109 172.1 mm to (185.3, 105.3), turned to -90 degrees
- moved C116 171.6 mm to (180.7, 105.3), turned to -90 degrees
- moved R112 171.4 mm to (186.9, 108.4), turned to 90 degrees
- moved J101 168.6 mm to (221.0, 85.2), turned to 90 degrees
- moved J103 167.9 mm to (210.9, 100.3), turned to 90 degrees
- moved R129 165.4 mm to (183.8, 108.4), turned to 90 degrees
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Connections:
- J103 pad 1: Net-(J103-Pad1) -> +24V
Routing:
- net +3V3: track 7.77 -> 29.3 mm, vias 0 -> 5
- net GND: track 22.8 -> 43.7 mm, vias 0 -> 10
- net /XIN: track 0.00 -> 8.97 mm
- net Net-(TP102-Pad1): track 0.00 -> 8.51 mm
- net Net-(J111-Pin_3): track 0.00 -> 7.95 mm
- net Net-(J111-Pin_2): track 0.00 -> 7.94 mm
- net Net-(R109-Pad2): track 0.00 -> 6.85 mm
- net Net-(J106-Pin_2): track 0.00 -> 6.77 mm
- net Net-(R124-Pad2): track 0.00 -> 6.76 mm
- net Net-(J107-Pin_2): track 0.00 -> 6.73 mm
- net /XOUT: track 0.00 -> 6.67 mm
- net Net-(R106-Pad2): track 0.00 -> 6.65 mm
- net Net-(R126-Pad2): track 0.00 -> 6.62 mm
- net Net-(J110-Pin_2): track 0.00 -> 6.60 mm
- net Net-(R125-Pad2): track 0.00 -> 6.53 mm
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Other:
- copper layers 2 -> 4
